Commit message: feat: add PR2 manipulation fixtures and update turtlebot3 EasyNav configs

File: robots_worlds/pr2/pr2.urdf (robot description, URDF)
Before this commit: robot pr2, 88 links, 87 joints
Links:
- link base_link: geometry collision mesh filename=file:///home/narinder/Documents/RobotLens-Workspace/RobotLe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; visual mesh filename=file:///home/narinder/Documents/RobotLens-Workspace/RobotLe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
- link bl_caster_l_wheel_link: geometry collision cylinder length=0.034 radius=0.074792; visual mesh filename=file:///home/narinder/Documents/RobotLens-Workspace/RobotLe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
- link bl_caster_r_wheel_link: geometry collision cylinder length=0.034 radius=0.074792; visual mesh filename=file:///home/narinder/Documents/RobotLens-Workspace/RobotLe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
- link bl_caster_rotation_link: geometry collision mesh filename=file:///home/narinder/Documents/RobotLens-Workspace/RobotLe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; visual mesh filename=file:///home/narinder/Documents/RobotLens-Workspace/RobotLe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
- link br_caster_l_wheel_link: geometry collision cylinder length=0.034 radius=0.074792; visual mesh filename=file:///home/narinder/Documents/RobotLens-Workspace/RobotLe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
- link br_caster_r_wheel_link: geometry collision cylinder length=0.034 radius=0.074792; visual mesh filename=file:///home/narinder/Documents/RobotLens-Workspace/RobotLe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
- link br_caster_rotation_link: geometry collision mesh filename=file:///home/narinder/Documents/RobotLens-Workspace/RobotLe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; visual mesh filename=file:///home/narinder/Documents/RobotLens-Workspace/RobotLe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
- link fl_caster_l_wheel_link: geometry collision cylinder length=0.034 radius=0.074792; visual mesh filename=file:///home/narinder/Documents/RobotLens-Workspace/RobotLe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
- link fl_caster_r_wheel_link: geometry collision cylinder length=0.034 radius=0.074792; visual mesh filename=file:///home/narinder/Documents/RobotLens-Workspace/RobotLe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
- link fl_caster_rotation_link: geometry collision mesh filename=file:///home/narinder/Documents/RobotLens-Workspace/RobotLe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; visual mesh filename=file:///home/narinder/Documents/RobotLens-Workspace/RobotLe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
- link fr_caster_l_wheel_link: geometry collision cylinder length=0.034 radius=0.074792; visual mesh filename=file:///home/narinder/Documents/RobotLens-Workspace/RobotLe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
- link fr_caster_r_wheel_link: geometry collision cylinder length=0.034 radius=0.074792; visual mesh filename=file:///home/narinder/Documents/RobotLens-Workspace/RobotLe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
- link fr_caster_rotation_link: geometry collision mesh filename=file:///home/narinder/Documents/RobotLens-Workspace/RobotLe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; visual mesh filename=file:///home/narinder/Documents/RobotLens-Workspace/RobotLe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
- link head_pan_link: geometry collision mesh filename=file:///home/narinder/Documents/RobotLens-Workspace/RobotLe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; visual mesh filename=file:///home/narinder/Documents/RobotLens-Workspace/RobotLe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
- link head_tilt_link: geometry collision mesh filename=file:///home/narinder/Documents/RobotLens-Workspace/RobotLe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; visual mesh filename=file:///home/narinder/Documents/RobotLens-Workspace/RobotLe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
- link l_elbow_flex_link: geometry collision mesh filename=file:///home/narinder/Documents/RobotLens-Workspace/RobotLe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; visual mesh filename=file:///home/narinder/Documents/RobotLens-Workspace/RobotLe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
- link l_forearm_link: geometry collision mesh filename=file:///home/narinder/Documents/RobotLens-Workspace/RobotLe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; visual mesh filename=file:///home/narinder/Documents/RobotLens-Workspace/RobotLe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
- link l_forearm_roll_link: geometry collision mesh filename=file:///home/narinder/Documents/RobotLens-Workspace/RobotLe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; visual mesh filename=file:///home/narinder/Documents/RobotLens-Workspace/RobotLe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
- link l_gripper_l_finger_link: geometry collision mesh filename=file:///home/narinder/Documents/RobotLens-Workspace/RobotLe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; visual mesh filename=file:///home/narinder/Documents/RobotLens-Workspace/RobotLe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
- link l_gripper_l_finger_tip_link: geometry collision mesh filename=file:///home/narinder/Documents/RobotLens-Workspace/RobotLe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; visual mesh filename=file:///home/narinder/Documents/RobotLens-Workspace/RobotLe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
- link l_gripper_palm_link: geometry collision mesh filename=file:///home/narinder/Documents/RobotLens-Workspace/RobotLe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; visual mesh filename=file:///home/narinder/Documents/RobotLens-Workspace/RobotLe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
- link l_gripper_r_finger_link: geometry collision mesh filename=file:///home/narinder/Documents/RobotLens-Workspace/RobotLe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; visual mesh filename=file:///home/narinder/Documents/RobotLens-Workspace/RobotLe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
- link l_gripper_r_finger_tip_link: geometry collision mesh filename=file:///home/narinder/Documents/RobotLens-Workspace/RobotLe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; visual mesh filename=file:///home/narinder/Documents/RobotLens-Workspace/RobotLe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
- link l_shoulder_lift_link: geometry collision mesh filename=file:///home/narinder/Documents/RobotLens-Workspace/RobotLe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; visual mesh filename=file:///home/narinder/Documents/RobotLens-Workspace/RobotLe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
- link l_shoulder_pan_link: geometry collision mesh filename=file:///home/narinder/Documents/RobotLens-Workspace/RobotLe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; visual mesh filename=file:///home/narinder/Documents/RobotLens-Workspace/RobotLe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
- link l_upper_arm_link: geometry collision mesh filename=file:///home/narinder/Documents/RobotLens-Workspace/RobotLe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; visual mesh filename=file:///home/narinder/Documents/RobotLens-Workspace/RobotLe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
- link l_upper_arm_roll_link: geometry collision mesh filename=file:///home/narinder/Documents/RobotLens-Workspace/RobotLe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; visual mesh filename=file:///home/narinder/Documents/RobotLens-Workspace/RobotLe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
- link l_wrist_flex_link: geometry collision mesh filename=file:///home/narinder/Documents/RobotLens-Workspace/RobotLe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; visual mesh filename=file:///home/narinder/Documents/RobotLens-Workspace/RobotLe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
- link l_wrist_roll_link: geometry collision mesh filename=file:///home/narinder/Documents/RobotLens-Workspace/RobotLe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; visual mesh filename=file:///home/narinder/Documents/RobotLens-Workspace/RobotLe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
- link laser_tilt_mount_link: geometry collision mesh filename=file:///home/narinder/Documents/RobotLens-Workspace/RobotLe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; visual mesh filename=file:///home/narinder/Documents/RobotLens-Workspace/RobotLe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
- link r_elbow_flex_link: geometry collision mesh filename=file:///home/narinder/Documents/RobotLens-Workspace/RobotLe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; visual mesh filename=file:///home/narinder/Documents/RobotLens-Workspace/RobotLe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
- link r_forearm_link: geometry collision mesh filename=file:///home/narinder/Documents/RobotLens-Workspace/RobotLe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; visual mesh filename=file:///home/narinder/Documents/RobotLens-Workspace/RobotLe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
- link r_forearm_roll_link: geometry collision mesh filename=file:///home/narinder/Documents/RobotLens-Workspace/RobotLe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; visual mesh filename=file:///home/narinder/Documents/RobotLens-Workspace/RobotLe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
- link r_gripper_l_finger_link: geometry collision mesh filename=file:///home/narinder/Documents/RobotLens-Workspace/RobotLe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; visual mesh filename=file:///home/narinder/Documents/RobotLens-Workspace/RobotLe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
- link r_gripper_l_finger_tip_link: geometry collision mesh filename=file:///home/narinder/Documents/RobotLens-Workspace/RobotLe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; visual mesh filename=file:///home/narinder/Documents/RobotLens-Workspace/RobotLe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
- link r_gripper_palm_link: geometry collision mesh filename=file:///home/narinder/Documents/RobotLens-Workspace/RobotLe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; visual mesh filename=file:///home/narinder/Documents/RobotLens-Workspace/RobotLe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
- link r_gripper_r_finger_link: geometry collision mesh filename=file:///home/narinder/Documents/RobotLens-Workspace/RobotLe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; visual mesh filename=file:///home/narinder/Documents/RobotLens-Workspace/RobotLe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
- link r_gripper_r_finger_tip_link: geometry collision mesh filename=file:///home/narinder/Documents/RobotLens-Workspace/RobotLe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; visual mesh filename=file:///home/narinder/Documents/RobotLens-Workspace/RobotLe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
- link r_shoulder_lift_link: geometry collision mesh filename=file:///home/narinder/Documents/RobotLens-Workspace/RobotLe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; visual mesh filename=file:///home/narinder/Documents/RobotLens-Workspace/RobotLe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
- link r_shoulder_pan_link: geometry collision mesh filename=file:///home/narinder/Documents/RobotLens-Workspace/RobotLe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; visual mesh filename=file:///home/narinder/Documents/RobotLens-Workspace/RobotLe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
- link r_upper_arm_link: geometry collision mesh filename=file:///home/narinder/Documents/RobotLens-Workspace/RobotLe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; visual mesh filename=file:///home/narinder/Documents/RobotLens-Workspace/RobotLe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
- link r_upper_arm_roll_link: geometry collision mesh filename=file:///home/narinder/Documents/RobotLens-Workspace/RobotLe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; visual mesh filename=file:///home/narinder/Documents/RobotLens-Workspace/RobotLe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
- link r_wrist_flex_link: geometry collision mesh filename=file:///home/narinder/Documents/RobotLens-Workspace/RobotLe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; visual mesh filename=file:///home/narinder/Documents/RobotLens-Workspace/RobotLe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
- link r_wrist_roll_link: geometry collision mesh filename=file:///home/narinder/Documents/RobotLens-Workspace/RobotLe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; visual mesh filename=file:///home/narinder/Documents/RobotLens-Workspace/RobotLe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
- link torso_lift_link: geometry collision mesh filename=file:///home/narinder/Documents/RobotLens-Workspace/RobotLe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; visual mesh filename=file:///home/narinder/Documents/RobotLens-Workspace/RobotLe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
